File: kicad/40106_oscillators.kicad_sch (KiCad schematic)
At the start: 19 parts, among them U1 40106

Commit message: update part numbers
Parts:
- U1: manf# (none) -> CD40106BE

Commit message: change pots
Parts:
- RV1, RV12, RV13, RV2, RV3, RV4: footprint elliot:Potentiometer_9mm_vertical_pcb_mount -> logic_noise:PTV09A4025FB104; manf# (none) -> PTV09A4025FB104
Changed lines of the file:
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@@
 			)
 		)
-		(property "Footprint" "elliot:Potentiometer_9mm_vertical_pcb_mount"
+		(property "Footprint" "logic_noise:PTV09A4025FB104"
 			(at 77.47 38.1 0)
 			(effects
@@
 			)
 		)
-		(property "manf#" ""
+		(property "manf#" "PTV09A4025FB104"
 			(at 77.47 38.1 0)
 			(effects
@@
 			)
 		)
-		(property "Footprint" "elliot:Potentiometer_9mm_vertical_pcb_mount"
+		(property "Footprint" "logic_noise:PTV09A4025FB104"
 			(at 77.47 83.82 0)
 			(effects
@@
 			)
 		)
-		(property "manf#" ""
+		(property "manf#" "PTV09A4025FB104"
 			(at 77.47 83.82 0)
 			(effects
@@
 			)
 		)
-		(property "Footprint" "elliot:Potentiometer_9mm_vertical_pcb_mount"
+		(property "Footprint" "logic_noise:PTV09A4025FB104"
 			(at 77.47 128.27 0)
 			(effects
@@
 			)
 		)
-		(property "manf#" ""
+		(property "manf#" "PTV09A4025FB104"
 			(at 77.47 128.27 0)
 			(effects
@@
 			)
 		)
-		(property "Footprint" "elliot:Potentiometer_9mm_vertical_pcb_mount"
+		(property "Footprint" "logic_noise:PTV09A4025FB104"
 			(at 76.2 160.02 0)
 			(effects
@@
 			)
 		)
-		(property "manf#" ""
+		(property "manf#" "PTV09A4025FB104"
 			(at 76.2 160.02 0)
 			(effects
@@
 			)
 		)
-		(property "Footprint" "elliot:Potentiometer_9mm_vertical_pcb_mount"
+		(property "Footprint" "logic_noise:PTV09A4025FB104"
 			(at 162.56 33.02 0)
 			(effects
@@
 			)
 		)
-		(property "manf#" ""
+		(property "manf#" "PTV09A4025FB104"
 			(at 162.56 33.02 0)
 			(effects
@@
 			)
 		)
-		(property "Footprint" "elliot:Potentiometer_9mm_vertical_pcb_mount"
+		(property "Footprint" "logic_noise:PTV09A4025FB104"
 			(at 162.56 90.17 0)
 			(effects
@@
 			)
 		)
-		(property "manf#" ""
+		(property "manf#" "PTV09A4025FB104"
 			(at 162.56 90.17 0)
 			(effects

Commit message: update stereo TRSS connector
Parts:
- C1, C2, C3, C4, C5, C6: manf# (none) -> Pines
- D1, D14, D15, D2, D3, D4: manf# (none) -> 1N4148

Commit message: update to kicad 9, add some comments and circuit changes
Parts:
- C1, C2, C3, C4, C5, C6: Comentarios (none) -> Es mejor soldar sólamente 2 de los 3 pines para mayor segur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; Orden (none) -> 99
- D1, D14, D15, D2, D3, D4, RV1, RV12, RV13, RV2, RV3, RV4, U1: Orden (none) -> 99
