File: kicad/bass_drum.kicad_sch (KiCad schematic)
At the start: 15 parts, among them U4 4069

Commit message: update part numbers
Parts:
- DECAY1: manf# (none) -> PTV09A-4025F-B104
- RV5: manf# (none) -> PDB182-K215K-503B1
- U4: manf# (none) -> CD4069UBE
Changed lines of the file:
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@@
 		(shape output)
 		(at 224.79 123.19 0)
+		(fields_autoplaced yes)
 		(effects
 			(font
@@
 		(shape output)
 		(at 176.53 49.53 0)
+		(fields_autoplaced yes)
 		(effects
 			(font
@@
 		(shape input)
 		(at 198.12 55.88 180)
+		(fields_autoplaced yes)
 		(effects
 			(font
@@
 		(shape input)
 		(at 135.89 31.75 180)
+		(fields_autoplaced yes)
 		(effects
 			(font
@@
 		(shape output)
 		(at 242.57 55.88 0)
+		(fields_autoplaced yes)
 		(effects
 			(font
@@
 		(shape input)
 		(at 30.48 71.12 180)
+		(fields_autoplaced yes)
 		(effects
 			(font
@@
 		(shape input)
 		(at 198.12 80.01 180)
+		(fields_autoplaced yes)
 		(effects
 			(font
@@
 		(shape output)
 		(at 176.53 31.75 0)
+		(fields_autoplaced yes)
 		(effects
 			(font
@@
 		(shape input)
 		(at 137.16 49.53 180)
+		(fields_autoplaced yes)
 		(effects
 			(font
@@
 		(shape output)
 		(at 245.11 80.01 0)
+		(fields_autoplaced yes)
 		(effects
 			(font
@@
 			)
 		)
+		(property "manf#" ""
+			(at 104.14 72.39 0)
+			(effects
+				(font
+					(size 1.27 1.27)
+				)
+				(hide yes)
+			)
+		)
 		(pin "1"
 		)
@@
 			)
 		)
+		(property "manf#" ""
+			(at 137.16 72.39 0)
+			(effects
+				(font
+					(size 1.27 1.27)
+				)
+				(hide yes)
+			)
+		)
 		(pin "1"
 		)
@@
 			)
 		)
+		(property "manf#" "PTV09A-4025F-B104 "
+			(at 120.65 78.74 0)
+			(effects
+				(font
+					(size 1.27 1.27)
+				)
+				(hide yes)
+			)
+		)
 		(pin "1"
 		)
@@
 			)
 		)
+		(property "manf#" "CD4069UBE"
+			(at 120.65 123.19 0)
+			(effects
+				(font
+					(size 1.27 1.27)
+				)
+				(hide yes)
+			)
+		)
 		(pin "14"
 		)
@@
 			)
 		)
+		(property "manf#" "CD4069UBE"
+			(at 181.61 123.19 0)
+			(effects
+				(font
+					(size 1.27 1.27)
+				)
+				(hide yes)
+			)
+		)
 		(pin "14"
 		)
@@
 			)
 		)
+		(property "manf#" ""
+			(at 181.61 114.3 0)
+			(effects
+				(font
+					(size 1.27 1.27)
+				)
+				(hide yes)
+			)
+		)
 		(pin "1"
 		)
@@
 			)
 		)
+		(property "manf#" ""
+			(at 158.75 123.19 0)
+			(effects
+				(font
+					(size 1.27 1.27)
+				)
+				(hide yes)
+			)
+		)
 		(pin "1"
 		)
@@
 			)
 		)
+		(property "manf#" ""
+			(at 180.34 105.41 0)
+			(effects
+				(font
+					(size 1.27 1.27)
+				)
+				(hide yes)
+			)
+		)
 		(pin "1"
 		)
@@
 			)
 		)
+		(property "manf#" "CD4069UBE"
+			(at 156.21 31.75 0)
+			(effects
+				(font
+					(size 1.27 1.27)
+				)
+				(hide yes)
+			)
+		)
 		(pin "14"
 		)
@@
 			)
 		)
+		(property "manf#" "CD4069UBE"
+			(at 156.21 49.53 0)
+			(effects
+				(font
+					(size 1.27 1.27)
+				)
+				(hide yes)
+			)
+		)
 		(pin "14"
 		)
@@
 			)
 		)
+		(property "manf#" "CD4069UBE"
+			(at 219.71 55.88 0)
+			(effects
+				(font
+					(size 1.27 1.27)
+				)
+				(hide yes)
+			)
+		)
 		(pin "14"
 		)
@@
 			)
 		)
+		(property "manf#" "CD4069UBE"
+			(at 219.71 80.01 0)
+			(effects
+				(font
+					(size 1.27 1.27)
+				)
+				(hide yes)
+			)
+		)
 		(pin "14"
 		)
@@
 			)
 		)
+		(property "manf#" ""
+			(at 115.57 107.95 0)
+			(effects
+				(font
+					(size 1.27 1.27)
+				)
+				(hide yes)
+			)
+		)
 		(pin "1"
 		)
@@
 			)
 		)
+		(property "manf#" ""
+			(at 123.19 107.95 0)
+			(effects
+				(font
+					(size 1.27 1.27)
+				)
+				(hide yes)
+			)
+		)
 		(pin "1"
 		)
@@
 			)
 		)
+		(property "manf#" ""
+			(at 53.34 80.01 0)
+			(effects
+				(font
+					(size 1.27 1.27)
+				)
+				(hide yes)
+			)
+		)
 		(pin "1"
 		)
@@
 			)
 		)
+		(property "manf#" ""
+			(at 40.64 71.12 0)
+			(effects
+				(font
+					(size 1.27 1.27)
+				)
+				(hide yes)
+			)
+		)
 		(pin "1"
 		)
@@
 			)
 		)
+		(property "manf#" ""
+			(at 63.5 71.12 0)
+			(effects
+				(font
+					(size 1.27 1.27)
+				)
+				(hide yes)
+			)
+		)
 		(pin "1"
 		)
@@
 			)
 		)
+		(property "manf#" "PDB182-K215K-503B1 "
+			(at 119.38 99.06 0)
+			(effects
+				(font
+					(size 1.27 1.27)
+				)
+				(hide yes)
+			)
+		)
 		(pin "1"
 		)
@@
 			)
 		)
+		(property "manf#" ""
+			(at 157.48 22.86 0)
+			(effects
+				(font
+					(size 1.27 1.27)
+				)
+				(hide yes)
+			)
+		)
 		(pin "1"
 		)
@@
 			(at 156.21 40.64 0)
 			(effects
+				(font
+					(size 1.27 1.27)
+				)
+				(hide yes)
+			)
+		)
+		(property "manf#" ""
+			(at 156.21 40.64 0)
+			(effects

Commit message: change pots
Parts:
- RV7, RV8: footprint elliot:Potentiometer_9mm_vertical_pcb_mount -> logic_noise:PTV09A4025FB104; manf# (none) -> PTV09A4025FB104
Changed lines of the file:
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@@
 			)
 		)
-		(property "Footprint" "elliot:Potentiometer_9mm_vertical_pcb_mount"
+		(property "Footprint" "logic_noise:PTV09A4025FB104"
 			(at 157.48 22.86 0)
 			(effects
@@
 			)
 		)
-		(property "manf#" ""
+		(property "manf#" "PTV09A4025FB104"
 			(at 157.48 22.86 0)
 			(effects
@@
 			)
 		)
-		(property "Footprint" "elliot:Potentiometer_9mm_vertical_pcb_mount"
+		(property "Footprint" "logic_noise:PTV09A4025FB104"
 			(at 156.21 40.64 0)
 			(effects
@@
 			)
 		)
-		(property "manf#" ""
+		(property "manf#" "PTV09A4025FB104"
 			(at 156.21 40.64 0)
 			(effects

Commit message: update resistors values
Parts:
- DECAY1: footprint elliot:Potentiometer_9mm_vertical_pcb_mount -> logic_noise:PTV09A4025FB104
- R3, R4: manf# (none) -> CF18JT100K
- RV5: footprint Potentiometers:Potentiometer_Alps-RK16-double -> Potentiometer_THT:Potentiometer_Alps_RK163_Dual_Horizontal; manf# PDB182-K215K-503B1 -> PTN16-A100230K1B2
Changed lines of the file:
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@@
 			)
 		)
-		(property "Footprint" "elliot:Potentiometer_9mm_vertical_pcb_mount"
+		(property "Footprint" "logic_noise:PTV09A4025FB104"
 			(at 120.65 78.74 0)
 			(effects
@@
 			)
 		)
-		(property "manf#" ""
+		(property "manf#" "CF18JT100K"
 			(at 181.61 114.3 0)
 			(effects
@@
 			)
 		)
-		(property "manf#" ""
+		(property "manf#" "CF18JT100K"
 			(at 158.75 123.19 0)
 			(effects
@@
 			)
 		)
-		(property "Footprint" "Potentiometers:Potentiometer_Alps-RK16-double"
+		(property "Footprint" "Potentiometer_THT:Potentiometer_Alps_RK163_Dual_Horizontal"
 			(at 119.38 99.06 0)
 			(effects
@@
 			)
 		)
-		(property "manf#" "PDB182-K215K-503B1 "
+		(property "manf#" "PTN16-A100230K1B2 "
 			(at 119.38 99.06 0)
 			(effects

Commit message: update stereo TRSS connector
Parts:
- C13, C14, C33, C34: manf# (none) -> C322C104M5U5TA
- C16: manf# (none) -> C322C103M5U5TA
- C19: manf# (none) -> C322C105M5U5TA
- D8, D9: manf# (none) -> 1N4148

Commit message: update to kicad 9, add some comments and circuit changes
Parts:
- C13, C14, C16, C19, C33, C34, D8, D9, DECAY1, R3, R4, RV5, RV7, RV8, U4: Orden (none) -> 99
