File: kicad/six_oscs.kicad_sch (KiCad schematic)
At the start: 13 parts, among them U3 40106

Commit message: update part numbers
Parts:
- U3: manf# (none) -> CD40106BE
Changed lines of the file:
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@@
 		(shape output)
 		(at 97.79 173.99 0)
+		(fields_autoplaced yes)
 		(effects
 			(font
@@
 		(shape output)
 		(at 88.9 87.63 0)
+		(fields_autoplaced yes)
 		(effects
 			(font
@@
 		(shape output)
 		(at 67.31 33.02 0)
+		(fields_autoplaced yes)
 		(effects
 			(font
@@
 		(shape output)
 		(at 67.31 119.38 0)
+		(fields_autoplaced yes)
 		(effects
 			(font
@@
 		(shape output)
 		(at 67.31 153.67 0)
+		(fields_autoplaced yes)
 		(effects
 			(font
@@
 		(shape output)
 		(at 67.31 67.31 0)
+		(fields_autoplaced yes)
 		(effects
 			(font
@@
 			)
 		)
+		(property "manf#" "CD40106BE"
+			(at 38.1 33.02 0)
+			(effects
+				(font
+					(size 1.27 1.27)
+				)
+				(hide yes)
+			)
+		)
 		(pin "1"
 		)
@@
 		(instances
 			(project "logic_noise_playground"
-				(path "/b9341db6-1cc2-4b11-8dd1-ce51623beade"
-					(reference "U3")
-					(unit 1)
-				)
 				(path "/b9341db6-1cc2-4b11-8dd1-ce51623beade/00000000-0000-0000-0000-0000554d4e92"
 					(reference "U3")
@@
 			)
 		)
+		(property "manf#" ""
+			(at 25.4 44.45 0)
+			(effects
+				(font
+					(size 1.27 1.27)
+				)
+				(hide yes)
+			)
+		)
 		(pin "2"
 		)
@@
 			)
 		)
+		(property "manf#" "CD40106BE"
+			(at 38.1 67.31 0)
+			(effects
+				(font
+					(size 1.27 1.27)
+				)
+				(hide yes)
+			)
+		)
 		(pin "1"
 		)
@@
 		(instances
 			(project "logic_noise_playground"
-				(path "/b9341db6-1cc2-4b11-8dd1-ce51623beade"
-					(reference "U3")
-					(unit 2)
-				)
 				(path "/b9341db6-1cc2-4b11-8dd1-ce51623beade/00000000-0000-0000-0000-0000554d4e92"
 					(reference "U3")
@@
 			)
 		)
+		(property "manf#" ""
+			(at 25.4 78.74 0)
+			(effects
+				(font
+					(size 1.27 1.27)
+				)
+				(hide yes)
+			)
+		)
 		(pin "1"
 		)
@@
 			)
 		)
+		(property "manf#" "CD40106BE"
+			(at 64.77 87.63 0)
+			(effects
+				(font
+					(size 1.27 1.27)
+				)
+				(hide yes)
+			)
+		)
 		(pin "1"
 		)
@@
 		(instances
 			(project "logic_noise_playground"
-				(path "/b9341db6-1cc2-4b11-8dd1-ce51623beade"
-					(reference "U3")
-					(unit 3)
-				)
 				(path "/b9341db6-1cc2-4b11-8dd1-ce51623beade/00000000-0000-0000-0000-0000554d4e92"
 					(reference "U3")
@@
 			)
 		)
+		(property "manf#" ""
+			(at 52.07 99.06 0)
+			(effects
+				(font
+					(size 1.27 1.27)
+				)
+				(hide yes)
+			)
+		)
 		(pin "1"
 		)
@@
 			)
 		)
+		(property "manf#" "CD40106BE"
+			(at 38.1 119.38 0)
+			(effects
+				(font
+					(size 1.27 1.27)
+				)
+				(hide yes)
+			)
+		)
 		(pin "1"
 		)
@@
 		(instances
 			(project "logic_noise_playground"
-				(path "/b9341db6-1cc2-4b11-8dd1-ce51623beade"
-					(reference "U3")
-					(unit 4)
-				)
 				(path "/b9341db6-1cc2-4b11-8dd1-ce51623beade/00000000-0000-0000-0000-0000554d4e92"
 					(reference "U3")
@@
 			)
 		)
+		(property "manf#" ""
+			(at 25.4 130.81 0)
+			(effects
+				(font
+					(size 1.27 1.27)
+				)
+				(hide yes)
+			)
+		)
 		(pin "1"
 		)
@@
 			)
 		)
+		(property "manf#" "CD40106BE"
+			(at 38.1 153.67 0)
+			(effects
+				(font
+					(size 1.27 1.27)
+				)
+				(hide yes)
+			)
+		)
 		(pin "1"
 		)
@@
 		(instances
 			(project "logic_noise_playground"
-				(path "/b9341db6-1cc2-4b11-8dd1-ce51623beade"
-					(reference "U3")
-					(unit 5)
-				)
 				(path "/b9341db6-1cc2-4b11-8dd1-ce51623beade/00000000-0000-0000-0000-0000554d4e92"
 					(reference "U3")
@@
 			)
 		)
+		(property "manf#" ""
+			(at 25.4 165.1 0)
+			(effects
+				(font
+					(size 1.27 1.27)
+				)
+				(hide yes)
+			)
+		)
 		(pin "1"
 		)
@@
 			)
 		)
+		(property "manf#" "CD40106BE"
+			(at 64.77 173.99 0)
+			(effects
+				(font
+					(size 1.27 1.27)
+				)
+				(hide yes)
+			)
+		)
 		(pin "1"
 		)
@@
 		(instances
 			(project "logic_noise_playground"
-				(path "/b9341db6-1cc2-4b11-8dd1-ce51623beade"
-					(reference "U3")
-					(unit 6)
-				)
 				(path "/b9341db6-1cc2-4b11-8dd1-ce51623beade/00000000-0000-0000-0000-0000554d4e92"
 					(reference "U3")
@@
 			)
 		)
+		(property "manf#" ""
+			(at 52.07 185.42 0)
+			(effects
+				(font
+					(size 1.27 1.27)
+				)
+				(hide yes)
+			)
+		)
 		(pin "1"
 		)
@@
 			)
 		)
+		(property "manf#" ""
+			(at 63.5 163.83 0)
+			(effects
+				(font
+					(size 1.27 1.27)
+				)
+				(hide yes)
+			)
+		)
 		(pin "1"
 		)
@@
 			)
 		)
+		(property "manf#" ""
+			(at 35.56 109.22 0)
+			(effects
+				(font
+					(size 1.27 1.27)
+				)
+				(hide yes)
+			)
+		)
 		(pin "1"
 		)
@@
 			)
 		)
+		(property "manf#" ""
+			(at 35.56 22.86 0)
+			(effects
+				(font
+					(size 1.27 1.27)
+				)
+				(hide yes)
+			)
+		)
 		(pin "1"
 		)
@@
 			)
 		)
+		(property "manf#" ""
+			(at 62.23 77.47 0)
+			(effects
+				(font
+					(size 1.27 1.27)
+				)
+				(hide yes)
+			)
+		)
 		(pin "1"
 		)
@@
 			)
 		)
+		(property "manf#" ""
+			(at 35.56 57.15 0)
+			(effects
+				(font
+					(size 1.27 1.27)
+				)
+				(hide yes)
+			)
+		)
 		(pin "1"
 		)
@@
 			(at 35.56 143.51 0)
 			(effects
+				(font
+					(size 1.27 1.27)
+				)
+				(hide yes)
+			)
+		)
+		(property "manf#" ""
+			(at 35.56 143.51 0)
+			(effects

Commit message: update resistors values
Parts:
- R14: manf# (none) -> CF14JT10K0
- R15: manf# (none) -> CF14JT33K0
- R16: manf# (none) -> CF14JT22K0
- R17: manf# (none) -> CF14JT47K0
- R18: manf# (none) -> CF14JT56K0
- R19: manf# (none) -> CF14JT39K0
Changed lines of the file:
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@@
 			)
 		)
-		(property "manf#" ""
+		(property "manf#" "CF14JT39K0"
 			(at 63.5 163.83 0)
 			(effects
@@
 			)
 		)
-		(property "manf#" ""
+		(property "manf#" "CF14JT47K0"
 			(at 35.56 109.22 0)
 			(effects
@@
 			)
 		)
-		(property "manf#" ""
+		(property "manf#" "CF14JT10K0"
 			(at 35.56 22.86 0)
 			(effects
@@
 			)
 		)
-		(property "manf#" ""
+		(property "manf#" "CF14JT22K0"
 			(at 62.23 77.47 0)
 			(effects
@@
 			)
 		)
-		(property "manf#" ""
+		(property "manf#" "CF14JT33K0"
 			(at 35.56 57.15 0)
 			(effects
@@
 			)
 		)
-		(property "manf#" ""
+		(property "manf#" "CF14JT56K0"
 			(at 35.56 143.51 0)
 			(effects

Commit message: update caps
Parts:
- C8: manf# (none) -> C322C104M5U5TA
Changed lines of the file:
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@@
 			)
 		)
-		(property "manf#" ""
+		(property "manf#" "C322C104M5U5TA"
 			(at 25.4 78.74 0)
 			(effects

Commit message: update stereo TRSS connector
Parts:
- C10, C11, C12, C7, C9: manf# (none) -> C322C104M5U5TA

Commit message: update to kicad 9, add some comments and circuit changes
Parts:
- C10, C11, C12, C7, C8, C9, U3: Orden (none) -> 99
- R14: value 10k -> 56k; Orden (none) -> 99
- R15: value 33k -> 47k; Orden (none) -> 99
- R16: value 22k -> 39k; Orden (none) -> 99
- R17: value 47k -> 33k; Orden (none) -> 99
- R18: value 56k -> 22k; Orden (none) -> 99
- R19: value 39k -> 10k; Orden (none) -> 99
