File: kicad/utility.kicad_sch (KiCad schematic)
At the start: 20 parts, among them P18 CONN_01X04, P33 CONN_01X04, P34 CONN_01X04, P35 CONN_01X04, P38 CONN_01X04, P39 CONN_01X04

Commit message: update resistors values
Parts:
- R10, R28: manf# (none) -> CF18JT100K
- R29, R30: manf# (none) -> CF14JT1K00
Changed lines of the file:
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@@
 			)
 		)
-		(property "manf#" ""
+		(property "manf#" "CF18JT100K"
 			(at 69.85 53.34 0)
 			(effects
@@
 			)
 		)
-		(property "manf#" ""
+		(property "manf#" "CF18JT100K"
 			(at 68.58 96.52 0)
 			(effects
@@
 			)
 		)
-		(property "manf#" ""
+		(property "manf#" "CF14JT1K00 "
 			(at 215.9 64.77 0)
 			(effects
@@
 			)
 		)
-		(property "manf#" ""
+		(property "manf#" "CF14JT1K00 "
 			(at 215.9 57.15 0)
 			(effects

Commit message: update caps
Parts:
- D21: manf# (none) -> NTE3144
- D22: manf# (none) -> NTE3145
Changed lines of the file:
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@@
 			)
 		)
-		(property "manf#" ""
+		(property "manf#" "NTE3144"
 			(at 204.47 57.15 0)
 			(effects
@@
 			)
 		)
-		(property "manf#" ""
+		(property "manf#" " NTE3145"
 			(at 204.47 64.77 0)
 			(effects

Commit message: update stereo TRSS connector
Parts:
- D10, D11, D18, D19, D20, D5, D6, D7: manf# (none) -> 1N4148
- P18, P33, P34, P35, P38, P39: manf# (none) -> Pines

Commit message: update to kicad 9, add some comments and circuit changes
Parts:
- D10, D11, D18, D19, D20, D21, D22, D5, D6, D7, P18, P33, P34, P35, P38, P39, R10, R28, R29, R30: Orden (none) -> 99
